File: ps2m.kicad_pcb (KiCad board)
At the start: 2 copper layers, 6 parts, among them P1 MOUSE_PORT, P2 CONN_01X06, U1 PIC16(L)F627-xxI/SS

Commit message: GND connection
Parts:
- P2: value CONN_01X06 -> MINI_DIN_6
Connections:
- P2 pad 7: (no net) -> GND
Routing:
- net GND: track 29.1 -> 47.7 mm
Changed lines of the file:
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@@
 (kicad_pcb (version 4) (host pcbnew 4.0.5)
   (general
-    (links 20)
-    (no_connects 1)
+    (links 23)
+    (no_connects 3)
     (area 0 0 0 0)
     (thickness 1.6)
     (drawings 4)
-    (tracks 143)
+    (tracks 151)
     (zones 0)
     (modules 6)
@@
   )
   (setup
-    (last_trace_width 0.2)
+    (last_trace_width 0.5)
     (user_trace_width 0.2)
     (user_trace_width 0.3)
@@
       (effects (font (size 1 1) (thickness 0.15)))
     )
-    (fp_text value CONN_01X06 (at 0 -1 180) (layer F.Fab)
+    (fp_text value MINI_DIN_6 (at 0 -1 180) (layer F.Fab)
       (effects (font (size 1 1) (thickness 0.15)))
     )
@@
     (fp_line (start -7 0) (end -7 3.5) (layer F.SilkS) (width 0.15))
     (fp_line (start -7 0) (end 7 0) (layer F.SilkS) (width 0.15))
-    (pad 7 thru_hole circle (at 0 4.7 270) (size 3 3) (drill 2.2) (layers *.Cu *.Mask))
-    (pad 7 smd rect (at -6 5.5 270) (size 3 2) (layers B.Cu F.Paste F.Mask))
-    (pad 7 smd rect (at 6 5.5 270) (size 3 2) (layers B.Cu F.Paste F.Mask))
+    (pad 7 thru_hole circle (at 0 4.7 270) (size 3 3) (drill 2.2) (layers *.Cu *.Mask)
+      (net 2 GND))
+    (pad 7 smd rect (at -6 5.5 270) (size 3 2) (layers B.Cu F.Paste F.Mask)
+      (net 2 GND))
+    (pad 7 smd rect (at 6 5.5 270) (size 3 2) (layers B.Cu F.Paste F.Mask)
+      (net 2 GND))
     (pad 1 thru_hole circle (at 1.3 8.5 270) (size 1.5 1.5) (drill 1) (layers *.Cu *.Mask)
       (net 10 /MINIDIN_1))
@@
   (segment (start 154.1 90.325) (end 152.875 90.325) (width 0.3) (layer B.Cu) (net 1))
   (segment (start 146.9 90.975) (end 148.075 90.975) (width 0.3) (layer B.Cu) (net 1))
+  (segment (start 152.4 100.4) (end 147.6 105.2) (width 0.5) (layer B.Cu) (net 2))
+  (segment (start 152.37 95.58) (end 152.37 100.37) (width 0.5) (layer F.Cu) (net 2))
+  (segment (start 152.37 100.37) (end 152.4 100.4) (width 0.5) (layer F.Cu) (net 2))
+  (segment (start 147.6 105.2) (end 147.6 106.8) (width 0.5) (layer F.Cu) (net 2))
+  (segment (start 147.6 106.8) (end 149.8 109) (width 0.5) (layer F.Cu) (net 2))
+  (segment (start 149.8 109) (end 151 109) (width 0.5) (layer F.Cu) (net 2))
+  (segment (start 145 108.2) (end 150.2 108.2) (width 0.5) (layer B.Cu) (net 2))
+  (segment (start 150.2 108.2) (end 151 109) (width 0.5) (layer B.Cu) (net 2))
+  (segment (start 157 108.2) (end 151.8 108.2) (width 0.5) (layer B.Cu) (net 2))
+  (segment (start 151.8 108.2) (end 151 109) (width 0.5) (layer B.Cu) (net 2))
   (segment (start 150.692081 93.592081) (end 151.477919 94.377919) (width 0.3) (layer B.Cu) (net 2))
   (segment (start 151.477919 94.377919) (end 152.37 94.377919) (width 0.3) (layer B.Cu) (net 2))
   (segment (start 148.317081 90.325) (end 150.692081 92.7) (width 0.3) (layer B.Cu) (net 2))
   (segment (start 150.692081 92.7) (end 150.692081 93.592081) (width 0.3) (layer B.Cu) (net 2))
-  (segment (start 152.4 100.4) (end 152.4 95.61) (width 0.3) (layer F.Cu) (net 2))
   (segment (start 152.4 95.61) (end 152.37 95.58) (width 0.3) (layer F.Cu) (net 2))
-  (segment (start 147.6 105.2) (end 152.4 100.4) (width 0.3) (layer B.Cu) (net 2))
   (via (at 152.4 100.4) (size 0.6) (drill 0.4) (layers F.Cu B.Cu) (net 2))
   (segment (start 156.4 92.6) (end 155.40001 93.59999) (width 0.2) (layer B.Cu) (net 2))

Commit message: Silkscreen
Other:
- board text added: "C1"
- board text added: "J1"
- board text added: "J3"
- board text added: "P1"
- board text added: "P2"
- board text added: "U1"
Changed lines of the file:
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@@
   (general
     (links 23)
-    (no_connects 3)
+    (no_connects 0)
     (area 0 0 0 0)
     (thickness 1.6)
-    (drawings 4)
+    (drawings 32)
     (tracks 151)
     (zones 0)
@@
   (layers
     (0 F.Cu signal)
-    (31 B.Cu signal)
+    (31 B.Cu signal hide)
     (32 B.Adhes user)
     (33 F.Adhes user)
     (34 B.Paste user)
     (35 F.Paste user)
-    (36 B.SilkS user)
-    (37 F.SilkS user)
+    (36 B.SilkS user hide)
+    (37 F.SilkS user hide)
     (38 B.Mask user)
     (39 F.Mask user)
     (40 Dwgs.User user)
     (41 Cmts.User user)
-    (42 Eco1.User user)
+    (42 Eco1.User user hide)
     (43 Eco2.User user)
     (44 Edge.Cuts user)
@@
     (47 F.CrtYd user)
     (48 B.Fab user hide)
-    (49 F.Fab user)
+    (49 F.Fab user hide)
   )
   (setup
@@
       (net 12 /JOY_3))
   )
+  (gr_text P1 (at 150.5 90) (layer Eco1.User)
+    (effects (font (size 1.5 1.5) (thickness 0.3)))
+  )
+  (gr_text P2 (at 151 112) (layer Eco1.User)
+    (effects (font (size 1.5 1.5) (thickness 0.3)))
+  )
+  (gr_text J3 (at 153.6 112) (layer Eco2.User)
+    (effects (font (size 1.2 1.2) (thickness 0.2)) (justify mirror))
+  )
+  (gr_text J1 (at 148.3 112) (layer Eco2.User)
+    (effects (font (size 1.2 1.2) (thickness 0.2)) (justify mirror))
+  )
+  (gr_line (start 148.6 104) (end 148.6 104.6) (layer Eco2.User) (width 0.2))
+  (gr_line (start 148.6 106.4) (end 148.6 105.8) (layer Eco2.User) (width 0.2))
+  (gr_line (start 150.9 106.4) (end 148.6 106.4) (layer Eco2.User) (width 0.2))
+  (gr_line (start 150.9 104) (end 150.9 106.4) (layer Eco2.User) (width 0.2))
+  (gr_line (start 148.6 104) (end 150.9 104) (layer Eco2.User) (width 0.2))
+  (gr_text U1 (at 150.5 90) (layer Eco2.User)
+    (effects (font (size 1.2 1.2) (thickness 0.2)) (justify mirror))
+  )
+  (gr_text C1 (at 156.3 93.4) (layer Eco2.User)
+    (effects (font (size 1.2 1.2) (thickness 0.2)) (justify mirror))
+  )
+  (gr_line (start 156.4 87.7) (end 157.2 87.7) (layer Eco2.User) (width 0.2))
+  (gr_line (start 156.8 88.1) (end 156.8 87.3) (layer Eco2.User) (width 0.2))
+  (gr_line (start 157.2 88.4) (end 155.6 88.4) (layer Eco2.User) (width 0.2))
+  (gr_line (start 157.2 92.4) (end 157.2 88.4) (layer Eco2.User) (width 0.2))
+  (gr_line (start 155.6 92.4) (end 157.2 92.4) (layer Eco2.User) (width 0.2))
+  (gr_line (start 155.6 92.3) (end 155.6 92.4) (layer Eco2.User) (width 0.2))
+  (gr_line (start 155.6 88.4) (end 155.6 92.3) (layer Eco2.User) (width 0.2))
+  (gr_line (start 144.2 99.8) (end 144.2 97) (layer Eco2.User) (width 0.2))
+  (gr_line (start 147 99.8) (end 144.2 99.8) (layer Eco2.User) (width 0.2))
+  (gr_line (start 147 97) (end 147 99.8) (layer Eco2.User) (width 0.2))
+  (gr_line (start 144.2 97) (end 147 97) (layer Eco2.User) (width 0.2))
+  (gr_circle (center 147.9 94.109901) (end 148.4 94.209901) (layer Eco2.User) (width 0.2))
+  (gr_line (start 152.8 86.3) (end 148.2 86.3) (layer Eco2.User) (width 0.2))
+  (gr_line (start 152.8 93.6) (end 152.8 86.3) (layer Eco2.User) (width 0.2))
+  (gr_line (start 149.1 93.6) (end 152.8 93.6) (layer Eco2.User) (width 0.2))
+  (gr_line (start 148.2 92.7) (end 149.1 93.6) (layer Eco2.User) (width 0.2))
+  (gr_line (start 148.2 86.3) (end 148.2 92.7) (layer Eco2.User) (width 0.2))
   (gr_line (start 144 113.5) (end 158 113.5) (layer Margin) (width 0.2))
   (gr_line (start 144 85.5) (end 158 85.5) (layer Margin) (width 0.2))
