File: ps2m.sch (KiCad schematic (older format))
At the start: 6 parts, among them P1 MOUSE_PORT, P2 MINI_DIN_6, U1 PIC16(L)F627-xxI/SS

Commit message: Part numbers for BOM
Parts:
- P1: bom_partno (none) -> L77SDE09SA4CH4R
- P2: bom_partno (none) -> KMDLX-6S-AS
- U1: bom_partno (none) -> PIC16F627A-I/SS
Changed lines of the file:
@@
 F 2 "kuro:DB9F-RA-TH-EUR" H 1050 2750 50  0001 C CNN
 F 3 "" H 1050 2750 50  0000 C CNN
+F 4 "L77SDE09SA4CH4R" H 1050 2750 60  0001 C CNN "bom_partno"
 	1    1050 2750
 	-1   0    0    -1
@@
 F 2 "Housings_SSOP:SSOP-20_5.3x7.2mm_Pitch0.65mm" H 4000 2750 50  0001 C CIN
 F 3 "" H 4000 2750 50  0000 C CNN
+F 4 "PIC16F627A-I/SS" H 4000 2750 60  0001 C CNN "bom_partno"
 	1    4000 2750
 	1    0    0    -1
@@
 F 1 "MINI_DIN_6" V 7500 2800 50  0000 C CNN
 F 2 "kuro:miniDIN-6-TH-Wrap" H 7400 2800 50  0001 C CNN
-F 3 "" H 7400 2800 50  0000 C CNN
+F 3 "http://www.kycon.com/Pub_Eng_Draw/KMDLX-XS-AS.PDF" H 7400 2800 50  0001 C CNN
+F 4 "KMDLX-6S-AS" H 7400 2800 60  0001 C CNN "bom_partno"
 	1    7400 2800
 	1    0    0    -1
